File: PCBs/LED/main.sch (EAGLE design)
At the start: 76 parts

Commit message: updated bom and schematic
Parts:
- C1, C10, C11, C12, C13, C14, C15, C16, C17, C18, C19, C2, C20, C21, C22, C23, C24, C25, C26, C27, C28, C29, C3, C30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: device Seeed-Capacitor:CERAMIC-100NF-25V-10%-X7R(0402) -> OPL_Capacitor:CERAMIC-100NF-50V-10%-X7R(0805)
